File: schematics/A500 14Mhz Accelerator.kicad_pcb (KiCad board)
At the start: 2 copper layers, 121.9 x 57.1 mm, 26 parts, among them J1 Speed Selector, U1 68000 Boardside, U10 74HC74, U2 68HC000 Socket, U3 74HC86, U4 74HC74, U5 74LS27, U6 74LS112, U7 74HC04, U8 74LS157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

Commit message: Add files via upload
Parts:
- C1, C10, C11, C12, C2, C3, C4, C5, C6, C7, C8, C9: footprint Capacitor_THT:C_Axial_L3.8mm_D2.6mm_P7.50mm_Horizontal -> Capacitor_THT:C_Axial_L5.1mm_D3.1mm_P7.50mm_Horizontal
- R1, R2, R3: footprint Resistor_THT:R_Axial_DIN0204_L3.6mm_D1.6mm_P5.08mm_Horizontal -> Resistor_THT:R_Axial_DIN0207_L6.3mm_D2.5mm_P7.62mm_Horizontal
- moved C11 94.8 mm to (96.5, 153.7)
- moved U2 92.9 mm to (114.0, 136.2)
- moved C9 86.5 mm to (192.4, 135.9)
- moved U7 86.5 mm to (188.6, 128.3)
- moved C12 84.3 mm to (111.3, 118.7), turned to 180 degrees
- moved C4 61.1 mm to (192.4, 123.2)
- moved U5 61.1 mm to (188.6, 115.6)
- moved C2 43.1 mm to (162.6, 138.4), turned to 90 degrees
- moved C1 41.6 mm to (165.7, 148.6), turned to 90 degrees
- moved C5 41.5 mm to (192.4, 110.5)
- moved U4 41.5 mm to (188.6, 102.9)
- moved U6 35.9 mm to (130.1, 144.8), turned to 180 degrees
- moved J1 33.2 mm to (160.7, 153.0)
- moved C6 32.8 mm to (192.4, 90.2)
- moved U3 32.8 mm to (188.6, 90.2)
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Routing:
- net /CPU_AS14: track 122.7 -> 25.2 mm
- net /CPU_CLK14: track 119.9 -> 30.2 mm
- net /CPU_VPA: track 44.6 -> 118.6 mm
- net /CPU_A5: track 96.2 -> 25.7 mm
- net /CPU_E: track 77.2 -> 140.8 mm, vias 0 -> 1
- net /CPU_A6: track 90.7 -> 28.0 mm
- net /CPU_A7: track 91.2 -> 28.7 mm
- net /CPU_VPA14: track 108.0 -> 50.0 mm, vias 1 -> 0
- net /GND: track 341.4 -> 397.2 mm
- net /CPU_A9: track 86.1 -> 30.8 mm
- net /CPU_A8: track 85.6 -> 30.8 mm
- net /CPU_A3: track 94.2 -> 46.0 mm
- net /CPU_D3: track 41.1 -> 88.9 mm, vias 1 -> 2
- net /A500 14Mhz Accelerator Sheet 2/_E_OUT: track 10.9 -> 58.0 mm
- net /CPU_A4: track 94.4 -> 47.6 mm
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Other:
- board size 121.9 x 57.1 mm -> 110 x 75 mm
- board text added: "1 2 3"
- board text added: "2 - 3 = 7 MHz"
- board text added: "68000 Clock Doubler - Adapted from Schematic by Livio Plos (C) 1992"
- board text added: "J1: 1 - 2 = 14MHz"
- board text removed: "14Mhz Accelerator (C) 1992 Livio Plos"

Commit message: Add files via upload
Parts:
- moved U1 82.0 mm to (87.0, 113.0), turned to 90 degrees
- moved U2 25.5 mm to (88.5, 136.1), turned to 90 degrees
- moved C12 0.25 mm to (111.3, 118.5)
Routing:
- net /CPU_A6: track 28.0 -> 116.0 mm
- net /CPU_D3: track 88.9 -> 24.6 mm, vias 2 -> 0
- net /CPU_VMA: track 101.6 -> 42.3 mm
- net /CPU_AS: track 126.5 -> 185.5 mm, vias 2 -> 1
- net /CPU_A5: track 25.7 -> 80.7 mm, vias 0 -> 1
- net /CPU_D4: track 80.0 -> 25.1 mm
- net /CPU_VPA: track 118.6 -> 69.0 mm, vias 0 -> 1
- net /CPU_A7: track 28.7 -> 76.2 mm, vias 0 -> 1
- net /CPU_A11: track 35.4 -> 79.6 mm, vias 0 -> 1
- net /CPU_D1: track 69.4 -> 27.2 mm
- net /CPU_D2: track 69.5 -> 27.5 mm
- net /CPU_CLK14: track 30.2 -> 70.2 mm, vias 0 -> 1
- net /CPU_A8: track 30.8 -> 70.3 mm, vias 0 -> 2
- net /CPU_A9: track 30.8 -> 70.1 mm
- net /CPU_D0: track 62.8 -> 32.9 mm
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